Commit message: Added ground truth tf publisher, updated URDF to follow proper coordinate conventions (#26)
* Update description and simulation configurations

* removed old xacro file

File: src/description/urdf/athena_drive.urdf.xacro (robot description, xacro)
@@ -28,11 +28,11 @@
   <!-- Contains description of drive -->
   <xacro:description/>
-  <xacro:imu_sensor parent="base_link">
-    <origin xyz="0 0 0.0" rpy="0 0 0"/>
+  <xacro:imu_sensor parent="base_footprint">
+    <origin xyz="0.0 0.0 0.0" rpy="0 0 0"/>
   </xacro:imu_sensor>
-  <xacro:gps_sensor parent="base_link">
-    <origin xyz="0 0 0.0" rpy="0 0 0"/>
+  <xacro:gps_sensor parent="base_footprint">
+    <origin xyz="0.0 0.0 0.0" rpy="0 0 0"/>
   </xacro:gps_sensor>
-  <xacro:ground_truth_odometry/>
+  <xacro:ground_truth_odometry robot_base_frame="base_footprint"/>
   <xacro:depth_camera parent_link="base_link">
       <origin xyz="0.75 0 -0.37" rpy="0 0 0"/>

File: src/description/urdf/athena_drive_description.urdf.xacro (robot description, xacro)
@@ -6,11 +6,6 @@
     <xacro:macro name="description">
         <link name="base_link">
-            <inertial>
-                <origin xyz="0.775305042176281 -0.0692748019047986 -0.475175318827691" rpy="0 0 0" />
-                <mass value="44.0454429414672" />
-                <inertia ixx="1.41725466889743" ixy="0.00803894609354262" ixz="-1.19304822311593E-17" iyy="1.33698338807128" iyz="1.62926079635059E-16" izz="2.58380655400253" />
-            </inertial>
-            <visual>
-                <origin xyz="0 0 0" rpy="0 0 0" />
+            <visual>
+                <origin xyz="-0.775305042176281 0.0692748019047986 0.475175318827691" rpy="0 0 -0.094743" />
                 <geometry>
                     <mesh filename="package://description/meshes/chassis_base_link.STL" />
@@ -21,5 +16,5 @@
             </visual>
             <collision>
-                <origin xyz="0 0 0" rpy="0 0 0" />
+                <origin xyz="-0.775305042176281 0.0692748019047986 0.475175318827691" rpy="0 0 -0.094743" />
                 <geometry>
                     <mesh filename="package://description/meshes/chassis_base_link.STL" />
@@ -50,5 +45,5 @@
         </link>
         <joint name="suspension_front_left_joint" type="fixed">
-            <origin xyz="0.61263 0.22146 -0.74592" rpy="1.5708 0 0.094743" />
+            <origin xyz="-.13 0.2355 -.26" rpy="1.5708 0 0" />
             <parent link="base_link" />
             <child link="suspension_front_left_link" />
@@ -284,5 +279,5 @@
         <link name="suspension_front_right_link">
             <inertial>
-                <origin xyz="0.0996575069633246 0.177857108210349 0.0120793884653498" rpy="0 0 0" />
+                <origin xyz="0.0 0.177857108210349 0.0120793884653498" rpy="0 0 0" />
                 <mass value="0.815137674139981" />
                 <inertia ixx="0.00362369286611303" ixy="2.10533763884314E-06" ixz="-1.88068045019413E-07" iyy="0.0343314249178962" iyz="-6.67186692298955E-08" izz="0.0378758255771416" />
@@ -305,5 +300,5 @@
         </link>
         <joint name="suspension_front_right_joint" type="fixed">
-            <origin xyz="0.66803 -0.36146 -0.74592" rpy="1.5708 0 0.094743" />
+            <origin xyz="-.13 -0.36146 -.26" rpy="1.5708 0 0" />
             <parent link="base_link" />
             <child link="suspension_front_right_link" />
@@ -362,5 +357,5 @@
         </link>
         <joint name="steer_fr_joint" type="revolute">
-            <origin xyz="0 0 0.059903" rpy="3.1416 0.094743 3.1416" />
+            <origin xyz="0 0 0.059903" rpy="3.1416 0.0 3.1416" />
             <parent link="swerve_mount_2_link" />
             <child link="steer_2_link" />
@@ -391,5 +386,5 @@
         </link>
         <joint name="wheel_bracket_2_joint" type="fixed">
-            <origin xyz="0.0225042151326936 -0.128534743589743 0.0550203250295025" rpy="0 0.0947430505373176 0" />
+            <origin xyz="0.0225042151326936 -0.128534743589743 0.0550203250295025" rpy="0 0.0 0" />
             <parent link="steer_2_link" />
             <child link="wheel_bracket_2_link" />
@@ -475,5 +470,5 @@
         </link>
         <joint name="steer_br_joint" type="revolute">
-            <origin xyz="0 0 0.0599025014000917" rpy="0 -0.0947430505373176 0" />
+            <origin xyz="0 0 0.0599025014000917" rpy="0 0.0 0" />
             <parent link="swerve_mount_3_link" />
             <child link="steer_3_link" />
@@ -504,5 +499,5 @@
         </link>
         <joint name="wheel_bracket_3_joint" type="fixed">
-            <origin xyz="-0.011719658421911 -0.128534743589743 0.0584684115770519" rpy="0 0.0947430505373176 0" />
+            <origin xyz="-0.011719658421911 -0.128534743589743 0.0584684115770519" rpy="0 0.0 0" />
             <parent link="steer_3_link" />
             <child link="wheel_bracket_3_link" />
@@ -537,4 +532,11 @@
             <axis xyz="0 0 1" />
         </joint>
+        <!-- Base footprint frame with inverted X and Y axes -->
+        <link name="base_footprint" />
+        <joint name="base_footprint_joint" type="fixed">
+            <origin xyz="0 0 0" rpy="0 0 3.14159265359" />
+            <parent link="base_footprint" />
+            <child link="base_link" />
+        </joint>
     </xacro:macro>
 </robot>

File: src/description/urdf/ground_truth_odom.xacro (robot description, xacro)
@@ -1,14 +1,12 @@
 <?xml version="1.0"?>
 <robot xmlns:xacro="http://www.ros.org/wiki/xacro">
-    <xacro:macro name="ground_truth_odometry" params="odom_frame:=odom robot_base_frame:=base_link odom_topic:=/odom/ground_truth update_rate:=50">
+    <xacro:macro name="ground_truth_odometry" params="robot_base_frame:=base_footprint odom_frame:=odom">
         <gazebo>
-            <plugin filename="ignition-gazebo-odometry-publisher-system" name="ignition::gazebo::systems::OdometryPublisher">
+            <plugin filename="libignition-gazebo-odometry-publisher-system.so"
+                    name="ignition::gazebo::systems::OdometryPublisher">
                 <odom_frame>${odom_frame}</odom_frame>
                 <robot_base_frame>${robot_base_frame}</robot_base_frame>
-                <odom_topic>${odom_topic}</odom_topic>
-                <odom_covariance_topic>${odom_topic}/covariance</odom_covariance_topic>
-                <tf_topic>${odom_topic}/tf</tf_topic>
-                <dimensions>3</dimensions>
-                <odom_publish_frequency>${update_rate}</odom_publish_frequency>
+                <odom_topic>/odom/ground_truth</odom_topic>
+                <odom_publish_frequency>50</odom_publish_frequency>
             </plugin>
         </gazebo>

File: src/description/urdf/imu.xacro (robot description, xacro)
@@ -24,4 +24,5 @@
                 <ign_frame_id>imu_link</ign_frame_id>
                 <plugin filename="libignition-gazebo-imu-system.so" name="ignition::gazebo::systems::Imu"/>
+                <initial_orientation_as_reference>false</initial_orientation_as_reference>
             </sensor>
         </gazebo>

Commit message: Depth Camera Visualization  (#27)
* added depth camera to urdf

* added rqt visualization for depth camera

---------

Co-authored-by: Mohammad Durrani <46766905+mdurrani808@users.noreply.github.com>

File: src/description/urdf/athena_drive.urdf.xacro (robot description, xacro)
@@ -35,6 +35,6 @@
   </xacro:gps_sensor>
   <xacro:ground_truth_odometry robot_base_frame="base_footprint"/>
-  <xacro:depth_camera parent_link="base_link">
-      <origin xyz="0.75 0 -0.37" rpy="0 0 0"/>
+  <xacro:depth_camera parent="base_footprint">
+      <origin xyz="0.0 0.0 0.1" rpy="0 0 0"/>
   </xacro:depth_camera>
   <xacro:if value="$(arg use_mock_hardware)">

File: src/description/urdf/depth_camera.xacro (robot description, xacro)
@@ -1,5 +1,5 @@
 <?xml version="1.0"?>
 <robot xmlns:xacro="http://www.ros.org/wiki/xacro">
-  <xacro:macro name="depth_camera" params="parent_link *origin">
+  <xacro:macro name="depth_camera" params="parent *origin">
     <link name="depth_camera_link">
       <visual>
@@ -18,16 +18,9 @@
         </geometry>
       </collision>
-      <inertial>
-        <mass value="0.072"/>
-        <origin xyz="0 0 0" rpy="0 0 0"/>
-        <inertia ixx="0.00001" ixy="0.0" ixz="0.0"
-                 iyy="0.00001" iyz="0.0"
-                 izz="0.00001"/>
-      </inertial>
     </link>
     <link name="depth_camera_optical_frame"/>
     <joint name="depth_camera_joint" type="fixed">
       <xacro:insert_block name="origin"/>
-      <parent link="${parent_link}"/>
+      <parent link="${parent}"/>
       <child link="depth_camera_link"/>
     </joint>
@@ -38,10 +31,11 @@
     </joint>
     <gazebo reference="depth_camera_link">
-      <sensor name="depth_camera" type="depth_camera">
+      <sensor name="depth_camera" type="depth">
         <always_on>1</always_on>
-        <update_rate>30</update_rate>
+        <update_rate>10</update_rate>
+        <visualize>true</visualize>
         <topic>depth_camera</topic>
         <camera name="depth_camera">
-          <horizontal_fov>1.047198</horizontal_fov>
+          <horizontal_fov>1.05</horizontal_fov>
           <image>
             <width>640</width>
@@ -53,6 +47,9 @@
             <far>10.0</far>
           </clip>
+          <depth_camera>
+	      	<output>points</output>
+	      </depth_camera>
         </camera>
-        <plugin filename="libgz-sim-sensors-system.so" name="gz::sim::systems::Sensors">
+        <plugin filename="libignition-gazebo-sensors-system.so" name="ignition::gazebo::systems::Sensors">
           <render_engine>ogre2</render_engine>
         </plugin>

Commit message: Added normal camera to URDF

File: src/description/urdf/athena_drive.urdf.xacro (robot description, xacro)
@@ -13,4 +13,5 @@
   <xacro:include filename="ground_truth_odom.xacro"/>
   <xacro:include filename="depth_camera.xacro"/>
+  <xacro:include filename="camera.xacro"/>
   <!-- Load robot's macro with parameters -->
   <!-- set prefix if multiple robots are used -->
@@ -38,4 +39,7 @@
       <origin xyz="0.0 0.0 0.1" rpy="0 0 0"/>
   </xacro:depth_camera>
+  <xacro:camera parent="base_footprint">
+    <origin xyz="0.0 0.0 0.15" rpy="0 0 0"/>
+  </xacro:camera>
   <xacro:if value="$(arg use_mock_hardware)">
     <xacro:athena_drive_ros2_control

Commit message: Get rid of old camera

File: src/description/urdf/athena_drive.urdf.xacro (robot description, xacro)
@@ -42,7 +42,4 @@
     <origin xyz=".5 0.1 0.1" rpy="0 0 0"/>
   </xacro:zed_camera_sensor>
-  <xacro:camera parent="base_footprint">
-    <origin xyz="0.0 0.0 0.15" rpy="0 0 0"/>
-  </xacro:camera>
   <xacro:if value="$(arg use_mock_hardware)">
     <xacro:athena_drive_ros2_control
